File: board/test-board.sch (KiCad schematic (older format))
At the start: 1 part

Commit message: More work on fleshing out test board
Parts:
- added D1, D2, D3, D4: LED, LEDs:LED_D5.0mm, symbol LED
- added J1, J2: Conn_01x01, Pin_Headers:Pin_Header_Straight_1x01_Pitch2.54mm, symbol Conn_01x01
- added J3: Conn_PWM, Pin_Headers:Pin_Header_Straight_1x04_Pitch2.54mm, symbol Conn_01x04
- added J5: Conn_UART, Pin_Headers:Pin_Header_Straight_1x03_Pitch2.54mm, symbol Conn_01x03
- added J6: Conn_SPI, Pin_Headers:Pin_Header_Straight_1x05_Pitch2.54mm, symbol Conn_01x05
- added J7: Conn_I2C, Pin_Headers:Pin_Header_Straight_1x04_Pitch2.54mm, symbol Conn_01x04
- added RN1: R_Pack04, nebrius-discrete:R_Array_Concave_4x2012.kicad_mod, symbol R_Pack04
- added SW1: SW_DPST_x2, symbol SW_DPST_x2
- J4: renamed from J?; footprint Pin_Headers:Pin_Header_Straight_2x20 -> Pin_Headers:Pin_Header_Straight_2x20_Pitch2.54mm
Connections:
- net at J4.10 ((RXD0)_GPIO15): now also J5.2 (Pin_2)
- net +3V3: now reaches J4.17 (3V3)
- net +3V3: now also J6.1 (Pin_1), J7.1 (Pin_1)
- net at J4.19 ((SPI_MOSI)_GPIO10): now also J6.3 (Pin_3)
- net at J4.21 ((SPI_MISO)_GPIO9): now also J6.2 (Pin_2)
- net at J4.23 ((SPI_SCLK)_GPIO11): now also J6.4 (Pin_4)
- net at J4.3 ((SDA1)_GPIO2): now also J7.2 (Pin_2)
- net at J4.35 (GPIO19): now also D1.2 (A), J3.1 (Pin_1)
- net at J4.37 (GPIO26): now also D4.2 (A), J3.4 (Pin_4)
- net at J4.38 (GPIO20): now also D2.2 (A), J3.2 (Pin_2)
- net GND: now reaches J4.39 (GND)
- net GND: now also J4.6 (GND), J1.1 (Pin_1), J2.1 (Pin_1), J5.3 (Pin_3), J6.5 (Pin_5), J7.4 (Pin_4), RN1.1 (R1.1), RN1.2 (R2.1), RN1.3 (R3.1), RN1.4 (R4.1), SW1.2 (B)
- net at J4.40 (GPIO21): now also D3.2 (A), J3.3 (Pin_3)
- net at J4.5 ((SCL1)_GPIO3): now also J7.3 (Pin_3)
- net at J4.7 ((GCLK)_GPIO4): now also SW1.1 (A)
- net at J4.8 ((TXD0)_GPIO14): now also J5.1 (Pin_1)
- new net: D1.1 (K), RN1.8 (R1.2)
- new net: D2.1 (K), RN1.7 (R2.2)
- new net: D3.1 (K), RN1.6 (R3.2)
- new net: D4.1 (K), RN1.5 (R4.2)
- no-connect marks 0 -> 25
